File: opena3xx-mcdu/kicad/opena3xx-mcdu/_autosave-opena3xx-mcdu.kicad_pcb (KiCad board)
At the start: 2 copper layers, 145.3 x 224.3 mm, 52 parts, among them J1 Conn_02x01, J2 Conn_02x01, J3 Conn_02x01, J4 Conn_02x01, J5 Conn_02x01, J6 Conn_02x01, J7 Conn_02x01, J8 Conn_02x01, J9 Conn_02x01, SW1 SW_MEC_5E, U1 MCP23017_SO, U2 MCP23017_SO, U3 MCP23017_SO, U4 MCP23017_SO, U5 MCP23017_SO

Commit message: MCDU Updates
Parts:
- moved SWL04 187.6 mm to (140.5, 88.7)
- moved D2 81.1 mm to (355.0, 150.6)
- moved SWR02 81.1 mm to (348.6, 149.6)
- moved R9 78.0 mm to (365.0, 146.6)
- moved R16 78.0 mm to (361.0, 151.0)
- moved SWR03 70.5 mm to (340.0, 149.6)
- moved SWL05 66.7 mm to (350.0, 138.5)
- moved J9 58.7 mm to (326.4, 152.6)
- moved SWL03 56.9 mm to (341.4, 138.5)
- moved R8 56.1 mm to (365.0, 143.3)
- moved D3 56.1 mm to (365.0, 140.0)
- moved R15 52.6 mm to (370.9, 140.3)
- moved R12 51.5 mm to (389.5, 122.0)
- moved R7 51.5 mm to (383.5, 125.3)
- moved SWR06 50.8 mm to (377.2, 110.0)
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
Commit message: Updates MCDU Schematic
Parts:
- removed SWL01, SWL02, SWL03, SWL04, SWL05, SWL06, SWR01, SWR02, SWR03, SWR04, SWR05, SWR06: TLL-6A, openaa3xx:TACTILE_LED_TH
- added R17: 220R, Resistor_SMD:R_1210_3225Metric_Pad1.30x2.65mm_HandSolder, F.Cu at (326.8, 100.8)
- added R18: 220R, Resistor_SMD:R_1210_3225Metric_Pad1.30x2.65mm_HandSolder, F.Cu at (308.9, 100.8)
- added R19: 220R, Resistor_SMD:R_1210_3225Metric_Pad1.30x2.65mm_HandSolder, F.Cu at (314.9, 100.8)
- added R20: 220R, Resistor_SMD:R_1210_3225Metric_Pad1.30x2.65mm_HandSolder, F.Cu at (320.8, 100.8)
- added SW10: TLL-6A, openaa3xx:TACTILE_LED_TH, F.Cu at (337.1, 66.0)
- added SW100: SW_MEC_5E, Button_Switch_THT:SW_TH_Tactile_Omron_B3F-10xx, F.Cu at (367.9, 89.1)
- added SW11: TLL-6A, openaa3xx:TACTILE_LED_TH, F.Cu at (328.4, 88.3)
- added SW12: TLL-6A, openaa3xx:TACTILE_LED_TH, F.Cu at (345.7, 66.0)
- added SW13: TLL-6A, openaa3xx:TACTILE_LED_TH, F.Cu at (337.1, 77.1)
- added SW14: TLL-6A, openaa3xx:TACTILE_LED_TH, F.Cu at (311.2, 66.0)
- added SW15: TLL-6A, openaa3xx:TACTILE_LED_TH, F.Cu at (345.7, 77.1)
- added SW16: TLL-6A, openaa3xx:TACTILE_LED_TH, F.Cu at (337.1, 88.3)
- added SW17: TLL-6A, openaa3xx:TACTILE_LED_TH, F.Cu at (354.3, 66.0)
- added SW18: TLL-6A, openaa3xx:TACTILE_LED_TH, F.Cu at (345.7, 88.3)
- added SW19: TLL-6A, openaa3xx:TACTILE_LED_TH, F.Cu at (362.9, 66.0)
- added SW2: TLL-6A, openaa3xx:TACTILE_LED_TH, F.Cu at (371.5, 77.1)
- added SW20: TLL-6A, openaa3xx:TACTILE_LED_TH, F.Cu at (354.3, 77.1)
- added SW21: TLL-6A, openaa3xx:TACTILE_LED_TH, F.Cu at (362.9, 77.1)
- added SW22: TLL-6A, openaa3xx:TACTILE_LED_TH, F.Cu at (354.3, 88.3)
- added SW23: TLL-6A, openaa3xx:TACTILE_LED_TH, F.Cu at (371.5, 66.0)
- added SW24: TLL-6A, openaa3xx:TACTILE_LED_TH, F.Cu at (362.9, 88.3)
- added SW3: TLL-6A, openaa3xx:TACTILE_LED_TH, F.Cu at (311.2, 77.1)
- added SW4: TLL-6A, openaa3xx:TACTILE_LED_TH, F.Cu at (319.8, 66.0)
- added SW5: TLL-6A, openaa3xx:TACTILE_LED_TH, F.Cu at (311.2, 88.3)
- added SW6: TLL-6A, openaa3xx:TACTILE_LED_TH, F.Cu at (328.4, 66.0)
- added SW7: TLL-6A, openaa3xx:TACTILE_LED_TH, F.Cu at (319.8, 77.1)
- added SW8: TLL-6A, openaa3xx:TACTILE_LED_TH, F.Cu at (328.4, 77.1)
- added SW9: TLL-6A, openaa3xx:TACTILE_LED_TH, F.Cu at (319.8, 88.3)
- SW1: value SW_MEC_5E -> TLL-6A; footprint Button_Switch_THT:SW_TH_Tactile_Omron_B3F-10xx -> openaa3xx:TACTILE_LED_TH
Connections:
- SW1 pad 1: GND -> /BUS0-0
- SW1 pad 3: RESET_SWITCH -> +12V
- SW1 pad 4: RESET_SWITCH -> Net-(SW1-Pad4)
- U1 pad 5: (no net) -> /BUS0-12
- U1 pad 6: (no net) -> /BUS0-13
- U1 pad 7: (no net) -> /BUS0-14
- U1 pad 8: (no net) -> /BUS0-15
- U2 pad 21: (no net) -> /BUS1-0
- U2 pad 22: (no net) -> /BUS1-1
- U2 pad 23: (no net) -> /BUS1-2
- U2 pad 24: (no net) -> /BUS1-3
- U2 pad 25: (no net) -> /BUS1-4
- U2 pad 26: (no net) -> /BUS1-5
- U2 pad 27: (no net) -> /BUS1-6
- U2 pad 28: (no net) -> /BUS1-7
