File: opena3xx-mcdu/kicad/opena3xx-mcdu/opena3xx-mcdu.sch (KiCad schematic (older format))
At the start: 84 parts, among them J1 Conn_02x01, J2 Conn_02x01, J3 Conn_02x01, J4 Conn_02x01, J5 Conn_02x01, J6 Conn_02x01, J7 Conn_02x01, J8 Conn_02x01, J9 Conn_02x01, SW1 TLL-6A, SW10 TLL-6A, SW100 SW_MEC_5E, SW11 TLL-6A, SW12 TLL-6A, SW13 TLL-6A, SW14 TLL-6A, SW15 TLL-6A, SW16 TLL-6A, SW17 TLL-6A, SW18 TLL-6A, SW19 TLL-6A, SW2 TLL-6A, SW20 TLL-6A, SW21 TLL-6A, SW22 TLL-6A, SW23 TLL-6A, SW24 TLL-6A, SW25 TLL-6A, SW26 TLL-6A, SW27 TLL-6A, SW28 TLL-6A, SW29 TLL-6A, SW3 TLL-6A, SW30 TLL-6A, SW31 TLL-6A, SW32 TLL-6A, SW33 TLL-6A, SW34 TLL-6A, SW35 TLL-6A, SW36 TLL-6A, SW4 TLL-6A, SW5 TLL-6A, SW6 TLL-6A, SW7 TLL-6A, SW8 TLL-6A, SW9 TLL-6A, U1 MCP23017_SO, U2 MCP23017_SO, U3 MCP23017_SO, U4 MCP23017_SO, U5 MCP23017_SO

Commit message: Completed MCDU Schematic v0.1
Parts:
- added D10: MCDU MENU - WHITE LED, Diode_SMD:D_1206_3216Metric_Pad1.42x1.75mm_HandSolder, symbol Device:LED
- added D11: FM - White LED, Diode_SMD:D_1206_3216Metric_Pad1.42x1.75mm_HandSolder, symbol Device:LED
- added D5: FM1 - Amber LED, Diode_SMD:D_1206_3216Metric_Pad1.42x1.75mm_HandSolder, symbol Device:LED
- added D6: FM2 - Amber LED, Diode_SMD:D_1206_3216Metric_Pad1.42x1.75mm_HandSolder, symbol Device:LED
- added D7: IND- Amber LED, Diode_SMD:D_1206_3216Metric_Pad1.42x1.75mm_HandSolder, symbol Device:LED
- added D8: RDY - Green LED, Diode_SMD:D_1206_3216Metric_Pad1.42x1.75mm_HandSolder, symbol Device:LED
- added D9: FAIL - Amber LED, Diode_SMD:D_1206_3216Metric_Pad1.42x1.75mm_HandSolder, symbol Device:LED
- added R25, R26, R27, R28, R29, R30, R31, R32, R33, R34, R35: 220R, Resistor_SMD:R_1210_3225Metric_Pad1.30x2.65mm_HandSolder, symbol Device:R_Small
- added R36: 470R, Resistor_SMD:R_1210_3225Metric_Pad1.30x2.65mm_HandSolder, symbol Device:R_Small
- added R37, R38, R39, R40, R41, R42, R43: 470R, Resistor_SMD:R_1206_3216Metric_Pad1.30x1.75mm_HandSolder, symbol Device:R_Small
- added SW37, SW38, SW39, SW40, SW41, SW42, SW43, SW44, SW45, SW46, SW47, SW48, SW49, SW50, SW51, SW52, SW53, SW54, SW55, SW56, SW57, SW58, SW59, SW60, SW61, SW62, SW63, SW64, SW65, SW66, SW67, SW68, SW69, SW70: TLL-6A, openaa3xx:TACTILE_LED_TH, symbol opena3xx-kicad:TLL-6A
Connections:
- net +12V: now also SW37.3, SW40.3, SW43.3, SW46.3, SW49.3, SW52.3, SW55.3, SW58.3, SW61.3, SW64.3, SW67.3, SW70.3
- net BUS2-10: now also SW43.1
- net BUS2-11: now also SW44.1
- net BUS2-12: now also SW45.1
- net BUS2-13: now also SW46.1
- net BUS2-14: now also SW47.1
- net BUS2-15: now also SW48.1
- net BUS2-4: now also SW37.1
- net BUS2-5: now also SW38.1
- net BUS2-6: now also SW39.1
- net BUS2-7: now also SW40.1
- net BUS2-8: now also SW41.1
- net BUS2-9: now also SW42.1
- net BUS3-0: now also SW49.1
- net BUS3-1: now also SW50.1
- net BUS3-10: now also SW59.1
- net BUS3-11: now also SW60.1
- net BUS3-12: now also SW61.1
- net BUS3-13: now also SW62.1
- net BUS3-14: now also SW63.1
- net BUS3-15: now also SW64.1
- net BUS3-2: now also SW51.1
- net BUS3-3: now also SW52.1
- net BUS3-4: now also SW53.1
- net BUS3-5: now also SW54.1
- net BUS3-6: now also SW55.1
- net BUS3-7: now also SW56.1
- net BUS3-8: now also SW57.1
- net BUS3-9: now also SW58.1
- net BUS4-0: now also SW65.1
- net BUS4-1: now also SW66.1
- net BUS4-10: now also D9.2 (A)
- net BUS4-11: now also D10.2 (A)
- net BUS4-12: now also D11.2 (A)
- net BUS4-2: now also SW67.1
- net BUS4-3: now also SW68.1
- net BUS4-4: now also SW69.1
- net BUS4-5: now also SW70.1
- net BUS4-6: now also D5.2 (A)
- net BUS4-7: now also D6.2 (A)
- net BUS4-8: now also D7.2 (A)
- net BUS4-9: now also D8.2 (A)
- net GND: now also R25.2, R26.2, R27.2, R28.2, R29.2, R30.2, R31.2, R32.2, R33.2, R34.2, R35.2, R36.2, R37.2, R38.2, R39.2, R40.2, R41.2, R42.2, R43.2, SW37.2, SW38.2, SW39.2, SW40.2, SW41.2, SW42.2, SW43.2, SW44.2, SW45.2, SW46.2, SW47.2, SW48.2, SW49.2, SW50.2, SW51.2, SW52.2, SW53.2, SW54.2, SW55.2, SW56.2, SW57.2, SW58.2, SW59.2, SW60.2, SW61.2, SW62.2, SW63.2, SW64.2, SW65.2, SW66.2, SW67.2, SW68.2, SW69.2, SW70.2
- net BUS4-13: no longer names the net of U5.6 (GPB5)
- net BUS4-14: no longer names the net of U5.7 (GPB6)
- net BUS4-15: no longer names the net of U5.8 (GPB7)
- new net: SW43.4, SW44.3
- new net: SW44.4, SW45.3
- new net: R27.1, SW45.4
- new net: SW46.4, SW47.3
- new net: SW47.4, SW48.3
- new net: R28.1, SW48.4
- new net: R26.1, SW42.4
- new net: SW41.4, SW42.3
- new net: SW40.4, SW41.3
- new net: R25.1, SW39.4
- new net: SW38.4, SW39.3
- new net: SW37.4, SW38.3
- new net: SW55.4, SW56.3
- new net: SW56.4, SW57.3
- new net: R31.1, SW57.4
- new net: SW58.4, SW59.3
- new net: SW59.4, SW60.3
- new net: R32.1, SW60.4
- new net: R30.1, SW54.4
- new net: SW53.4, SW54.3
- new net: SW52.4, SW53.3
- new net: R29.1, SW51.4
- new net: SW50.4, SW51.3
- new net: SW49.4, SW50.3
- new net: SW67.4, SW68.3
- new net: SW68.4, SW69.3
- new net: R35.1, SW69.4
- new net: R36.1, SW70.4
- new net: R34.1, SW66.4
- new net: SW65.4, SW66.3
- new net: SW64.4, SW65.3
- new net: R33.1, SW63.4
- new net: SW62.4, SW63.3
- new net: SW61.4, SW62.3
- new net: D5.1 (K), R37.1
- new net: D6.1 (K), R38.1
- new net: D7.1 (K), R39.1
- new net: D8.1 (K), R40.1
- new net: D9.1 (K), R41.1
- new net: D10.1 (K), R42.1
- new net: D11.1 (K), R43.1
- no-connect marks 30 -> 33
Other:
- note added: "Annunciators Lights"
- note added: "MCDU ALPHABET KEYS\n"

Commit message: WIP PCB Layout process for MCDU - ICs and connectors
Parts:
- SW1, SW10, SW11, SW12, SW13, SW14, SW15, SW16, SW17, SW18, SW19, SW2, SW20, SW21, SW22, SW23, SW24, SW25, SW26, SW27, SW28, SW29, SW3, SW30, SW31, SW32, SW33, SW34, SW35, SW36, SW37, SW38, SW39, SW4, SW40, SW41, SW42, SW43, SW44, SW45, SW46, SW47, SW48, SW49, SW5, SW50, SW51, SW52, SW53, SW54, SW55, SW56, SW57, SW58, SW59, SW6, SW60, SW61, SW62, SW63, SW64, SW65, SW66, SW67, SW68, SW69, SW7, SW70, SW8, SW9: symbol opena3xx-kicad:TLL-6A -> opena3xx-mcdu-rescue:TLL-6A-opena3xx-kicad

Commit message: Updated PCB MCDU v0.1
Parts:
- removed J1, J2: Conn_02x01, Connector_PinHeader_2.54mm:PinHeader_1x02_P2.54mm_Vertical, symbol Connector_Generic:Conn_02x01
- removed J8, J9: Conn_02x01, TerminalBlock:TerminalBlock_bornier-2_P5.08mm, symbol Connector_Generic:Conn_02x01
- added J5: Conn_02x01, TerminalBlock:TerminalBlock_bornier-2_P5.08mm, symbol Connector_Generic:Conn_02x01
- added R?: 220R, Resistor_SMD:R_1210_3225Metric_Pad1.30x2.65mm_HandSolder, symbol Device:R_Small
- added SW71, SW72: TLL-6A, openaa3xx:TACTILE_LED_TH, symbol opena3xx-mcdu-rescue:TLL-6A-opena3xx-kicad
- added SW73: SW_MEC_5E, Button_Switch_THT:SW_TH_Tactile_Omron_B3F-10xx, symbol Switch:SW_MEC_5E
- renumbered J3 to J1, J4 to J2, J6 to J3, J7 to J4
Connections:
- net +12V: now also SW71.3
- net GND: now also R?.2
- new net: J5.1 (Pin_1), SW73.1, SW73.2
- new net: J5.2 (Pin_2), SW73.3 (K), SW73.4 (A)
- new net: SW71.4, SW72.3
- new net: R?.1, SW72.4
Changed lines of the file:
@@
 $Comp
 L Connector_Generic:Conn_02x01 J1
-U 1 1 63B465A7
-P 8325 11150
-F 0 "J1" H 8375 11367 50  0000 C CNN
-F 1 "Conn_02x01" H 8375 11276 50  0000 C CNN
-F 2 "Connector_PinHeader_2.54mm:PinHeader_1x02_P2.54mm_Vertical" H 8325 11150 50  0001 C CNN
-F 3 "~" H 8325 11150 50  0001 C CNN
-	1    8325 11150
-	1    0    0    -1
-$EndComp
-$Comp
-L Connector_Generic:Conn_02x01 J2
-U 1 1 63B47049
-P 8325 11525
-F 0 "J2" H 8375 11742 50  0000 C CNN
-F 1 "Conn_02x01" H 8375 11651 50  0000 C CNN
-F 2 "Connector_PinHeader_2.54mm:PinHeader_1x02_P2.54mm_Vertical" H 8325 11525 50  0001 C CNN
-F 3 "~" H 8325 11525 50  0001 C CNN
-	1    8325 11525
-	1    0    0    -1
-$EndComp
-$Comp
-L Connector_Generic:Conn_02x01 J3
 U 1 1 63B4C595
 P 9225 11150
-F 0 "J3" H 9275 11367 50  0000 C CNN
+F 0 "J1" H 9275 11367 50  0000 C CNN
 F 1 "Conn_02x01" H 9275 11276 50  0000 C CNN
 F 2 "TerminalBlock:TerminalBlock_bornier-2_P5.08mm" H 9225 11150 50  0001 C CNN
@@
 $EndComp
 $Comp
-L power:+5V #PWR0143
-U 1 1 63BA0E89
-P 7950 10900
-F 0 "#PWR0143" H 7950 10750 50  0001 C CNN
-F 1 "+5V" H 7965 11073 50  0000 C CNN
-F 2 "" H 7950 10900 50  0001 C CNN
-F 3 "" H 7950 10900 50  0001 C CNN
-	1    7950 10900
-	1    0    0    -1
-$EndComp
-$Comp
 L power:+5V #PWR0144
 U 1 1 63BA22F1
@@
 $EndComp
 Wire Wire Line
-	8125 11150 7950 11150
-Wire Wire Line
-	7950 11150 7950 10900
-Wire Wire Line
-	8125 11525 7950 11525
-Wire Wire Line
-	7950 11525 7950 11150
-Connection ~ 7950 11150
-Wire Wire Line
 	8925 10925 8925 11150
 Wire Wire Line
@@
 Connection ~ 8925 11150
 $Comp
-L power:GND #PWR0145
-U 1 1 63CF7D16
-P 8750 11725
-F 0 "#PWR0145" H 8750 11475 50  0001 C CNN
-F 1 "GND" H 8755 11552 50  0000 C CNN
-F 2 "" H 8750 11725 50  0001 C CNN
-F 3 "" H 8750 11725 50  0001 C CNN
-	1    8750 11725
-	1    0    0    -1
-$EndComp
-$Comp
 L power:GND #PWR0146
 U 1 1 63CF9021
@@
 $EndComp
 Wire Wire Line
-	8750 11725 8750 11525
-Wire Wire Line
-	8750 11525 8625 11525
-Wire Wire Line
-	8750 11525 8750 11150
-Wire Wire Line
-	8750 11150 8625 11150
-Connection ~ 8750 11525
-Wire Wire Line
 	9650 11725 9650 11525
 Wire Wire Line
@@
 Connection ~ 9650 11525
 $Comp
-L Connector_Generic:Conn_02x01 J4
+L Connector_Generic:Conn_02x01 J2
 U 1 1 63B4C59B
 P 9225 11525
-F 0 "J4" H 9275 11742 50  0000 C CNN
+F 0 "J2" H 9275 11742 50  0000 C CNN
 F 1 "Conn_02x01" H 9275 11651 50  0000 C CNN
 F 2 "TerminalBlock:TerminalBlock_bornier-2_P5.08mm" H 9225 11525 50  0001 C CNN
@@
 Supply Terminal Blocks\n5V & 12V Variable for Backlight\n
 $Comp
-L Switch:SW_MEC_5E SW100
-U 1 1 60A66F25
-P 3525 1625
-F 0 "SW100" H 3525 2010 50  0000 C CNN
-F 1 "SW_MEC_5E" H 3525 1919 50  0000 C CNN
-F 2 "Button_Switch_THT:SW_TH_Tactile_Omron_B3F-10xx" H 3525 1925 50  0001 C CNN
-F 3 "http://www.apem.com/int/index.php?controller=attachment&id_attachment=1371" H 3525 1925 50  0001 C CNN
-	1    3525 1625
-	1    0    0    -1
-$EndComp
-$Comp
 L power:+5V #PWR0147
 U 1 1 60A6870F
@@
 Wire Wire Line
 	3125 1900 3125 1525
-Wire Wire Line
-	3125 1525 3250 1525
 Text GLabel 3800 2000 0    50   Output ~ 0
 RESET_SWITCH
@@
 	3775 4950 3425 4950
 Wire Wire Line
-	3325 1625 3250 1625
-Wire Wire Line
-	3250 1625 3250 1525
-Connection ~ 3250 1525
-Wire Wire Line
-	3250 1525 3325 1525
-Wire Wire Line
 	3725 1625 3825 1625
 Connection ~ 3825 1625
@@
 MCDU RIGHT SIDE KEYS\n
 $Comp
-L Connector_Generic:Conn_02x01 J6
+L Connector_Generic:Conn_02x01 J3
 U 1 1 60F73FB9
 P 10125 11150
-F 0 "J6" H 10175 11367 50  0000 C CNN
+F 0 "J3" H 10175 11367 50  0000 C CNN
 F 1 "Conn_02x01" H 10175 11276 50  0000 C CNN
 F 2 "TerminalBlock:TerminalBlock_bornier-2_P5.08mm" H 10125 11150 50  0001 C CNN
@@
 Connection ~ 10550 11525
 $Comp
-L Connector_Generic:Conn_02x01 J7
+L Connector_Generic:Conn_02x01 J4
 U 1 1 60F73FD5
 P 10125 11525
-F 0 "J7" H 10175 11742 50  0000 C CNN
+F 0 "J4" H 10175 11742 50  0000 C CNN
 F 1 "Conn_02x01" H 10175 11651 50  0000 C CNN
 F 2 "TerminalBlock:TerminalBlock_bornier-2_P5.08mm" H 10125 11525 50  0001 C CNN
@@
 	1    0    0    -1
 $EndComp
-$Comp
-L Connector_Generic:Conn_02x01 J8
-U 1 1 6105AECB
-P 10975 11150
-F 0 "J8" H 11025 11367 50  0000 C CNN
-F 1 "Conn_02x01" H 11025 11276 50  0000 C CNN
-F 2 "TerminalBlock:TerminalBlock_bornier-2_P5.08mm" H 10975 11150 50  0001 C CNN
-F 3 "~" H 10975 11150 50  0001 C CNN
-	1    10975 11150
-	1    0    0    -1
-$EndComp
-Wire Wire Line
-	10675 11150 10775 11150
-Wire Wire Line
-	10775 11525 10675 11525
-Wire Wire Line
-	10675 11525 10675 11150
-Connection ~ 10675 11150
-$Comp
-L power:GND #PWR0128
-U 1 1 6105AED5
-P 11400 11725
-F 0 "#PWR0128" H 11400 11475 50  0001 C CNN
-F 1 "GND" H 11405 11552 50  0000 C CNN
-F 2 "" H 11400 11725 50  0001 C CNN
-F 3 "" H 11400 11725 50  0001 C CNN
-	1    11400 11725
-	1    0    0    -1
-$EndComp
-Wire Wire Line
-	11400 11725 11400 11525
-Wire Wire Line
-	11400 11525 11275 11525
-Wire Wire Line
-	11400 11525 11400 11150
-Wire Wire Line
-	11400 11150 11275 11150
-Connection ~ 11400 11525
-$Comp
-L Connector_Generic:Conn_02x01 J9
-U 1 1 6105AEE0
-P 10975 11525
-F 0 "J9" H 11025 11742 50  0000 C CNN
-F 1 "Conn_02x01" H 11025 11651 50  0000 C CNN
-F 2 "TerminalBlock:TerminalBlock_bornier-2_P5.08mm" H 10975 11525 50  0001 C CNN
-F 3 "~" H 10975 11525 50  0001 C CNN
-	1    10975 11525
-	1    0    0    -1
-$EndComp
-$Comp
-L power:+12V #PWR0129
-U 1 1 6105AEE6
-P 10675 10925
-F 0 "#PWR0129" H 10675 10775 50  0001 C CNN
-F 1 "+12V" H 10690 11098 50  0000 C CNN
-F 2 "" H 10675 10925 50  0001 C CNN
-F 3 "" H 10675 10925 50  0001 C CNN
-	1    10675 10925
-	1    0    0    -1
-$EndComp
-Wire Wire Line
-	10675 10925 10675 11150
 Wire Notes Line
 	11650 10375 11650 11975
@@
 NoConn ~ 19925 2575
 NoConn ~ 19925 2675
+Wire Wire Line
+	3250 1525 3325 1525
+Connection ~ 3250 1525
+Wire Wire Line
+	3250 1625 3250 1525
+Wire Wire Line
+	3325 1625 3250 1625
+Wire Wire Line
+	3125 1525 3250 1525
+$Comp
+L Switch:SW_MEC_5E SW100
+U 1 1 60A66F25
+P 3525 1625
+F 0 "SW100" H 3525 2010 50  0000 C CNN
+F 1 "SW_MEC_5E" H 3525 1919 50  0000 C CNN
+F 2 "Button_Switch_THT:SW_TH_Tactile_Omron_B3F-10xx" H 3525 1925 50  0001 C CNN
+F 3 "http://www.apem.com/int/index.php?controller=attachment&id_attachment=1371" H 3525 1925 50  0001 C CNN
+	1    3525 1625
+	1    0    0    -1
+$EndComp
+$Comp
+L Switch:SW_MEC_5E SW73
+U 1 1 60C5FAF8
+P 14525 11150
+F 0 "SW73" H 14525 11535 50  0000 C CNN
+F 1 "SW_MEC_5E" H 14525 11444 50  0000 C CNN
+F 2 "Button_Switch_THT:SW_TH_Tactile_Omron_B3F-10xx" H 14525 11450 50  0001 C CNN
+F 3 "http://www.apem.com/int/index.php?controller=attachment&id_attachment=1371" H 14525 11450 50  0001 C CNN
+	1    14525 11150
+	1    0    0    -1
+$EndComp
+$Comp
+L Connector_Generic:Conn_02x01 J5
+U 1 1 60F77B96
+P 14475 10625
+F 0 "J5" H 14525 10842 50  0000 C CNN
+F 1 "Conn_02x01" H 14525 10751 50  0000 C CNN
+F 2 "TerminalBlock:TerminalBlock_bornier-2_P5.08mm" H 14475 10625 50  0001 C CNN
+F 3 "~" H 14475 10625 50  0001 C CNN
+	1    14475 10625
+	1    0    0    -1
+$EndComp
+Wire Wire Line
+	14275 10625 14175 10625
+Wire Wire Line
+	14175 10625 14175 11050
+Wire Wire Line
+	14175 11050 14325 11050
+Wire Wire Line
+	14775 10625 14825 10625
+Wire Wire Line
+	14825 10625 14825 11050
+Wire Wire Line
+	14825 11050 14725 11050
+Wire Wire Line
+	14175 11050 14175 11150
+Wire Wire Line
+	14175 11150 14325 11150
+Connection ~ 14175 11050
+Wire Wire Line
+	14725 11150 14825 11150
+Wire Wire Line
+	14825 11150 14825 11050
+Connection ~ 14825 11050
+$Comp
+L opena3xx-mcdu-rescue:TLL-6A-opena3xx-kicad SW71
+U 1 1 61EBD1D6
+P 15925 10625
+F 0 "SW71" H 16000 10830 50  0000 C CNN
+F 1 "TLL-6A" H 16000 10739 50  0000 C CNN
+F 2 "openaa3xx:TACTILE_LED_TH" H 16000 10648 50  0001 C CNN
+F 3 "https://eu.mouser.com/datasheet/2/910/312_TL-6-1571269.pdf" H 15925 10675 50  0001 C CNN
+F 4 "BRT" H 15925 10625 50  0000 C CNN "MCDU IO Name"
+	1    15925 10625
+	1    0    0    -1
+$EndComp
+$Comp
+L opena3xx-mcdu-rescue:TLL-6A-opena3xx-kicad SW72
+U 1 1 61F8A2B8
+P 16875 10625
+F 0 "SW72" H 16950 10830 50  0000 C CNN
+F 1 "TLL-6A" H 16950 10739 50  0000 C CNN
+F 2 "openaa3xx:TACTILE_LED_TH" H 16950 10648 50  0001 C CNN
+F 3 "https://eu.mouser.com/datasheet/2/910/312_TL-6-1571269.pdf" H 16875 10675 50  0001 C CNN
+F 4 "DIM" H 16875 10625 50  0000 C CNN "MCDU IO Name"
+	1    16875 10625
+	1    0    0    -1
+$EndComp
+Wire Wire Line
+	16275 10925 16675 10925
+$Comp
+L Device:R_Small R?
+U 1 1 6278A1A9
+P 17450 11125
+F 0 "R?" H 17509 11171 50  0000 L CNN
+F 1 "220R" H 17509 11080 50  0000 L CNN
+F 2 "Resistor_SMD:R_1210_3225Metric_Pad1.30x2.65mm_HandSolder" H 17450 11125 50  0001 C CNN
+F 3 "~" H 17450 11125 50  0001 C CNN
+	1    17450 11125
+	1    0    0    -1
+$EndComp
+Wire Wire Line
+	17225 10925 17450 10925
+Wire Wire Line
+	17450 10925 17450 11025
+$Comp
+L power:GND #PWR?
+U 1 1 628589E0
+P 17450 11425
+F 0 "#PWR?" H 17450 11175 50  0001 C CNN
+F 1 "GND" H 17455 11252 50  0000 C CNN
+F 2 "" H 17450 11425 50  0001 C CNN
+F 3 "" H 17450 11425 50  0001 C CNN
+	1    17450 11425
+	1    0    0    -1
+$EndComp
+Wire Wire Line
+	17450 11225 17450 11425
+$Comp
+L power:+12V #PWR?
+U 1 1 6292907A
+P 15500 10825
+F 0 "#PWR?" H 15500 10675 50  0001 C CNN
+F 1 "+12V" H 15515 10998 50  0001 C CNN
+F 2 "" H 15500 10825 50  0001 C CNN
+F 3 "" H 15500 10825 50  0001 C CNN
+	1    15500 10825
+	1    0    0    -1
+$EndComp
+Wire Wire Line
+	15500 10825 15500 10925
+Wire Wire Line
+	15500 10925 15725 10925
 Wire Bus Line
 	20850 5125 20850 10300
