File: opena3xx-mcdu/kicad/opena3xx-mcdu/opena3xx-mcdu.sch (KiCad schematic (older format))
At the start: 145 parts, among them J1 Conn_02x01, J2 Conn_02x01, J3 Conn_02x01, J4 Conn_02x01, J5 Conn_02x01, SW1 TLL-6A, SW10 TLL-6A, SW100 SW_MEC_5E, SW11 TLL-6A, SW12 TLL-6A, SW13 TLL-6A, SW14 TLL-6A, SW15 TLL-6A, SW16 TLL-6A, SW17 TLL-6A, SW18 TLL-6A, SW19 TLL-6A, SW2 TLL-6A, SW20 TLL-6A, SW21 TLL-6A, SW22 TLL-6A, SW23 TLL-6A, SW24 TLL-6A, SW25 TLL-6A, SW26 TLL-6A, SW27 TLL-6A, SW28 TLL-6A, SW29 TLL-6A, SW3 TLL-6A, SW30 TLL-6A, SW31 TLL-6A, SW32 TLL-6A, SW33 TLL-6A, SW34 TLL-6A, SW35 TLL-6A, SW36 TLL-6A, SW37 TLL-6A, SW38 TLL-6A, SW39 TLL-6A, SW4 TLL-6A, SW40 TLL-6A, SW41 TLL-6A, SW42 TLL-6A, SW43 TLL-6A, SW44 TLL-6A, SW45 TLL-6A, SW46 TLL-6A, SW47 TLL-6A, SW48 TLL-6A, SW49 TLL-6A, SW5 TLL-6A, SW50 TLL-6A, SW51 TLL-6A, SW52 TLL-6A, SW53 TLL-6A, SW54 TLL-6A, SW55 TLL-6A, SW56 TLL-6A, SW57 TLL-6A, SW58 TLL-6A, SW59 TLL-6A, SW6 TLL-6A, SW60 TLL-6A, SW61 TLL-6A, SW62 TLL-6A, SW63 TLL-6A, SW64 TLL-6A, SW65 TLL-6A, SW66 TLL-6A, SW67 TLL-6A, SW68 TLL-6A, SW69 TLL-6A, SW7 TLL-6A, SW70 TLL-6A, SW71 TLL-6A, SW72 TLL-6A, SW73 SW_MEC_5E, SW8 TLL-6A, SW9 TLL-6A, U1 MCP23017_SO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

Commit message: Finalised Layour for MCDU PCB v 0.1
Parts:
- removed SW73: SW_MEC_5E, Button_Switch_THT:SW_TH_Tactile_Omron_B3F-10xx, symbol Switch:SW_MEC_5E
- added J7: Conn_02x01, TerminalBlock:TerminalBlock_bornier-2_P5.08mm, symbol Connector_Generic:Conn_02x01
- gave numbers to parts that had none: 1
- renumbered J5 to J6
Connections:
- net at J6.1 (Pin_1): now also SW71.1
- net at J6.2 (Pin_2): now also SW71.2
- net at SW72.1: now also J7.1 (Pin_1)
- net at SW72.2: now also J7.2 (Pin_2)
Other:
- moved on the sheet: J6
Changed lines of the file:
@@
 $EndComp
 $Comp
-L Switch:SW_MEC_5E SW73
-U 1 1 60C5FAF8
-P 14525 11150
-F 0 "SW73" H 14525 11535 50  0000 C CNN
-F 1 "SW_MEC_5E" H 14525 11444 50  0000 C CNN
-F 2 "Button_Switch_THT:SW_TH_Tactile_Omron_B3F-10xx" H 14525 11450 50  0001 C CNN
-F 3 "http://www.apem.com/int/index.php?controller=attachment&id_attachment=1371" H 14525 11450 50  0001 C CNN
-	1    14525 11150
+L Connector_Generic:Conn_02x01 J6
+U 1 1 60F77B96
+P 15950 11475
+F 0 "J6" H 16000 11692 50  0000 C CNN
+F 1 "Conn_02x01" H 16000 11601 50  0000 C CNN
+F 2 "TerminalBlock:TerminalBlock_bornier-2_P5.08mm" H 15950 11475 50  0001 C CNN
+F 3 "~" H 15950 11475 50  0001 C CNN
+	1    15950 11475
 	1    0    0    -1
 $EndComp
-$Comp
-L Connector_Generic:Conn_02x01 J5
-U 1 1 60F77B96
-P 14475 10625
-F 0 "J5" H 14525 10842 50  0000 C CNN
-F 1 "Conn_02x01" H 14525 10751 50  0000 C CNN
-F 2 "TerminalBlock:TerminalBlock_bornier-2_P5.08mm" H 14475 10625 50  0001 C CNN
-F 3 "~" H 14475 10625 50  0001 C CNN
-	1    14475 10625
-	1    0    0    -1
-$EndComp
-Wire Wire Line
-	14275 10625 14175 10625
-Wire Wire Line
-	14175 10625 14175 11050
-Wire Wire Line
-	14175 11050 14325 11050
-Wire Wire Line
-	14775 10625 14825 10625
-Wire Wire Line
-	14825 10625 14825 11050
-Wire Wire Line
-	14825 11050 14725 11050
-Wire Wire Line
-	14175 11050 14175 11150
-Wire Wire Line
-	14175 11150 14325 11150
-Connection ~ 14175 11050
-Wire Wire Line
-	14725 11150 14825 11150
-Wire Wire Line
-	14825 11150 14825 11050
-Connection ~ 14825 11050
 $Comp
 L opena3xx-mcdu-rescue:TLL-6A-opena3xx-kicad SW71
@@
 	16275 10925 16675 10925
 $Comp
-L Device:R_Small R?
+L Device:R_Small R44
 U 1 1 6278A1A9
 P 17450 11125
-F 0 "R?" H 17509 11171 50  0000 L CNN
+F 0 "R44" H 17509 11171 50  0000 L CNN
 F 1 "220R" H 17509 11080 50  0000 L CNN
 F 2 "Resistor_SMD:R_1210_3225Metric_Pad1.30x2.65mm_HandSolder" H 17450 11125 50  0001 C CNN
@@
 	17450 10925 17450 11025
 $Comp
-L power:GND #PWR?
+L power:GND #PWR0128
 U 1 1 628589E0
 P 17450 11425
-F 0 "#PWR?" H 17450 11175 50  0001 C CNN
+F 0 "#PWR0128" H 17450 11175 50  0001 C CNN
 F 1 "GND" H 17455 11252 50  0000 C CNN
 F 2 "" H 17450 11425 50  0001 C CNN
@@
 	17450 11225 17450 11425
 $Comp
-L power:+12V #PWR?
+L power:+12V #PWR0129
 U 1 1 6292907A
 P 15500 10825
-F 0 "#PWR?" H 15500 10675 50  0001 C CNN
+F 0 "#PWR0129" H 15500 10675 50  0001 C CNN
 F 1 "+12V" H 15515 10998 50  0001 C CNN
 F 2 "" H 15500 10825 50  0001 C CNN
@@
 Wire Wire Line
 	15500 10925 15725 10925
+$Comp
+L Connector_Generic:Conn_02x01 J7
+U 1 1 62AD3D1C
+P 16900 11475
+F 0 "J7" H 16950 11692 50  0000 C CNN
+F 1 "Conn_02x01" H 16950 11601 50  0000 C CNN
+F 2 "TerminalBlock:TerminalBlock_bornier-2_P5.08mm" H 16900 11475 50  0001 C CNN
+F 3 "~" H 16900 11475 50  0001 C CNN
+	1    16900 11475
+	1    0    0    -1
+$EndComp
+Wire Wire Line
+	15750 11475 15625 11475
+Wire Wire Line
+	15625 11475 15625 10825
+Wire Wire Line
+	15625 10825 15725 10825
+Wire Wire Line
+	16250 11475 16400 11475
+Wire Wire Line
+	16400 11475 16400 10825
+Wire Wire Line
+	16400 10825 16275 10825
+Wire Wire Line
+	16550 10825 16550 11475
+Wire Wire Line
+	16550 11475 16700 11475
+Wire Wire Line
+	17200 11475 17275 11475
+Wire Wire Line
+	17275 11475 17275 10825
+Wire Wire Line
+	17275 10825 17225 10825
+Wire Wire Line
+	16550 10825 16675 10825
 Wire Bus Line
 	20850 5125 20850 10300
